File: trumpet_schematic/trumpet_schematic.kicad_sch (KiCad schematic)
At the start: 17 parts, among them J1 LCD, Q1 NPN, SW1 SW_Push, SW10 SW_Push, SW2 SW_Push, SW3 SW_Push, SW4 SW_Push, SW5 SW_Push, SW6 SW_Push, SW7 SW_Push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

Commit message: save
Parts:
- added 20Ω: R, symbol Device:R
Connections:
- net at Q1.1 (C): now also 20Ω.1; no longer R1.2
- new net: 20Ω.2, R1.2
Other:
- moved on the sheet: Q1, R2
Changed lines of the file:
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@@
+		)
+	)
+	(wire
+		(pts
+			(xy 95.25 91.44) (xy 95.25 99.06)
+		)
+		(stroke
+			(width 0)
+			(type default)
 		)
 	)
@@
 	(wire
 		(pts
-			(xy 57.15 102.87) (xy 73.66 102.87)
+			(xy 41.91 110.49) (xy 58.42 110.49)
 		)
 		(stroke
@@
 	(wire
 		(pts
-			(xy 95.25 107.95) (xy 95.25 127)
+			(xy 80.01 115.57) (xy 80.01 134.62)
 		)
 		(stroke
@@
 	(wire
 		(pts
+			(xy 80.01 99.06) (xy 82.55 99.06)
+		)
+		(stroke
+			(width 0)
+			(type default)
+		)
+	)
+	(wire
+		(pts
 			(xy 152.4 91.44) (xy 157.48 91.44)
 		)
@@
 	(wire
 		(pts
-			(xy 95.25 91.44) (xy 95.25 97.79)
+			(xy 80.01 99.06) (xy 80.01 105.41)
 		)
 		(stroke
@@
 	(wire
 		(pts
+			(xy 90.17 99.06) (xy 95.25 99.06)
+		)
+		(stroke
+			(width 0)
+			(type default)
+		)
+	)
+	(wire
+		(pts
 			(xy 138.43 106.68) (xy 177.8 106.68)
 		)
@@
 	(wire
 		(pts
-			(xy 81.28 102.87) (xy 87.63 102.87)
+			(xy 66.04 110.49) (xy 72.39 110.49)
 		)
 		(stroke
@@
 	)
 	(label "P2.4"
-		(at 57.15 102.87 180)
+		(at 41.91 110.49 180)
 		(effects
 			(font
@@
 	)
 	(label "GND"
-		(at 95.25 127 180)
+		(at 80.01 134.62 180)
 		(effects
 			(font
@@
 	)
 	(symbol
+		(lib_id "Device:R")
+		(at 86.36 99.06 90)
+		(unit 1)
+		(exclude_from_sim no)
+		(in_bom yes)
+		(on_board yes)
+		(dnp no)
+		(fields_autoplaced yes)
+		(property "Reference" "20Ω"
+			(at 86.36 92.71 90)
+			(effects
+				(font
+					(size 1.27 1.27)
+				)
+			)
+		)
+		(property "Value" "R"
+			(at 86.36 95.25 90)
+			(effects
+				(font
+					(size 1.27 1.27)
+				)
+			)
+		)
+		(property "Footprint" ""
+			(at 86.36 100.838 90)
+			(effects
+				(font
+					(size 1.27 1.27)
+				)
+				(hide yes)
+			)
+		)
+		(property "Datasheet" "~"
+			(at 86.36 99.06 0)
+			(effects
+				(font
+					(size 1.27 1.27)
+				)
+				(hide yes)
+			)
+		)
+		(property "Description" "Resistor"
+			(at 86.36 99.06 0)
+			(effects
+				(font
+					(size 1.27 1.27)
+				)
+				(hide yes)
+			)
+		)
+		(pin "2"
+		)
+		(pin "1"
+		)
+		(instances
+			(project ""
+				(path "/72e6d7f3-c76a-4c03-a31b-775dd92d8425"
+					(reference "20Ω")
+					(unit 1)
+				)
+			)
+		)
+	)
+	(symbol
 		(lib_id "Switch:SW_Push")
 		(at 229.87 135.89 0)
@@
 	(symbol
 		(lib_id "Device:R")
-		(at 77.47 102.87 90)
+		(at 62.23 110.49 90)
 		(unit 1)
 		(exclude_from_sim no)
@@
 		(fields_autoplaced yes)
 		(property "Reference" "R2"
-			(at 77.47 96.52 90)
+			(at 62.23 104.14 90)
 			(effects
 				(font
@@
 		)
 		(property "Value" "20Ω"
-			(at 77.47 99.06 90)
+			(at 62.23 106.68 90)
 			(effects
 				(font
@@
 		)
 		(property "Footprint" ""
-			(at 77.47 104.648 90)
+			(at 62.23 112.268 90)
 			(effects
 				(font
@@
 		)
 		(property "Datasheet" "~"
-			(at 77.47 102.87 0)
+			(at 62.23 110.49 0)
 			(effects
 				(font
@@
 		)
 		(property "Description" "Resistor"
-			(at 77.47 102.87 0)
+			(at 62.23 110.49 0)
 			(effects
 				(font
@@
 	(symbol
 		(lib_id "Simulation_SPICE:NPN")
-		(at 92.71 102.87 0)
+		(at 77.47 110.49 0)
 		(unit 1)
 		(exclude_from_sim no)
@@
 		(fields_autoplaced yes)
 		(property "Reference" "Q1"
-			(at 97.79 101.5999 0)
+			(at 82.55 109.2199 0)
 			(effects
 				(font
@@
 		)
 		(property "Value" "NPN"
-			(at 97.79 104.1399 0)
+			(at 82.55 111.7599 0)
 			(effects
 				(font
@@
 		)
 		(property "Footprint" ""
-			(at 156.21 102.87 0)
+			(at 140.97 110.49 0)
 			(effects
 				(font
@@
 		)
 		(property "Datasheet" "https://ngspice.sourceforge.io/docs/ngspice-html-manual/manual.xhtml#cha_BJTs"
-			(at 156.21 102.87 0)
+			(at 140.97 110.49 0)
 			(effects
 				(font
@@
 		)
 		(property "Description" "Bipolar transistor symbol for simulation only, substrate tied to the emitter"
-			(at 92.71 102.87 0)
+			(at 77.47 110.49 0)
 			(effects
 				(font
@@
 		)
 		(property "Sim.Device" "NPN"
-			(at 92.71 102.87 0)
+			(at 77.47 110.49 0)
 			(effects
 				(font
@@
 		)
 		(property "Sim.Type" "GUMMELPOON"
-			(at 92.71 102.87 0)
+			(at 77.47 110.49 0)
 			(effects
 				(font
@@
 		)
 		(property "Sim.Pins" "1=C 2=B 3=E"
-			(at 92.71 102.87 0)
-			(effects
-				(font
+			(at 77.47 110.49 0)
+			(effects
+				(font

Commit message: recent save
still needs comments and headers etc
Other:
- note added: "E"
- note added: "LCD"
- note added: "RS"
- note added: "Speaker"
Changed lines of the file:
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@@
+		)
+	)
+	(text "LCD"
+		(exclude_from_sim no)
+		(at 227.33 94.234 0)
+		(effects
+			(font
+				(size 1.27 1.27)
+			)
 		)
 	)
@@
 		)
 	)
+	(text "RS"
+		(exclude_from_sim no)
+		(at 227.584 101.6 0)
+		(effects
+			(font
+				(size 1.27 1.27)
+			)
+		)
+	)
 	(text "NOTES\n"
 		(exclude_from_sim no)
 		(at 203.2 115.57 0)
+		(effects
+			(font
+				(size 1.27 1.27)
+			)
+		)
+	)
+	(text "Speaker"
+		(exclude_from_sim no)
+		(at 226.822 88.9 0)
 		(effects
 			(font
@@
 		(effects
 			(font
+				(size 1.27 1.27)
+			)
+		)
+	)
+	(text "E"
+		(exclude_from_sim no)
+		(at 227.33 97.79 0)
+		(effects
+			(font
